File: atmel_ice_adapter.kicad_pcb (KiCad board)
At the start: 2 copper layers, 5 parts, among them J1 Conn_02x05_Odd_Even, J2 Conn_02x03_Odd_Even, J3 Conn_02x03_Odd_Even, J4 Conn_02x05_Odd_Even, J5 Conn_02x10_Odd_Even

Commit message: update foot print & layout
Parts:
- J1: footprint Connector_PinSocket_1.27mm:PinSocket_2x05_P1.27mm_Vertical -> Connector_PinHeader_1.27mm:PinHeader_2x05_P1.27mm_Vertical
- J2: footprint Connector_PinHeader_1.27mm:PinHeader_2x03_P1.27mm_Vertical -> Connector_PinSocket_1.27mm:PinSocket_2x03_P1.27mm_Horizontal
- J3: footprint Connector_PinHeader_2.54mm:PinHeader_2x03_P2.54mm_Vertical -> Connector_PinSocket_2.54mm:PinSocket_2x03_P2.54mm_Horizontal
- J4: footprint Connector_PinHeader_2.54mm:PinHeader_2x05_P2.54mm_Vertical -> Connector_PinSocket_2.54mm:PinSocket_2x05_P2.54mm_Horizontal
- J5: footprint Connector_PinHeader_2.54mm:PinHeader_2x10_P2.54mm_Vertical -> Connector_PinSocket_2.54mm:PinSocket_2x10_P2.54mm_Horizontal
- moved J4 25.7 mm to (101.6, 86.4)
- moved J1 25.5 mm to (104.1, 74.3)
- moved J2 24.4 mm to (125.7, 74.9), turned to 180 degrees
- moved J3 21.6 mm to (91.4, 71.1)
- moved J5 4.57 mm to (118.1, 67.3), turned to 270 degrees
Connections:
- J5 pad 10: Net-(J5-Pad10) -> /PIN9
- J5 pad 12: Net-(J5-Pad12) -> /PIN9
- J5 pad 18: Net-(J5-Pad18) -> /PIN5
- J5 pad 20: Net-(J5-Pad20) -> /PIN5
- J5 pad 4: Net-(J5-Pad4) -> /PIN3
- J5 pad 6: Net-(J5-Pad6) -> /PIN3
Other:
- board outline added: 51.6 x 41.9 mm

Commit message: update layout
Parts:
- moved J2 0.64 mm to (125.1, 74.9)
- moved J3 0.64 mm to (92.1, 71.1)
- moved J4 0.64 mm to (101.6, 85.7)
- moved J5 0.63 mm to (118.1, 67.9)
Other:
- board size 51.6 x 41.9 mm -> 51.1 x 41.9 mm

Commit message: update layout
Parts:
- moved J2 64.1 mm to (188.0, 87.6)
- moved J4 62.7 mm to (162.6, 100.3)
- moved J1 62.3 mm to (165.1, 87.0)
- moved J5 61.9 mm to (179.1, 78.7)
- moved J3 60.4 mm to (151.1, 83.8)
Other:
- board size 51.1 x 41.9 mm -> 54 x 44.5 mm
- net class Default: clearance 0.2 -> 0.1524; trace_width 0.25 -> 0.254; via_dia 0.8 -> 0.6096; via_drill 0.4 -> 0.3048
- rule trace_clearance: 0.2 -> 0.1524
- rule trace_min: 0.2 -> 0.127
- rule via_min_size: 0.4 -> 0.6

Commit message: auto routing
Routing:
- net /PIN9: track 0.00 -> 89.8 mm
- net /PIN4: track 0.00 -> 88.7 mm
- net /PIN6: track 0.00 -> 86.5 mm
- net /PIN3: track 0.00 -> 79.2 mm
- net /PIN2: track 0.00 -> 72.6 mm
- net /PIN1: track 0.00 -> 71.1 mm
- net /PIN5: track 0.00 -> 53.8 mm
- net /PIN7: track 0.00 -> 49.2 mm
- net /PIN8: track 0.00 -> 34.3 mm
- net /PIN10: track 0.00 -> 30.9 mm

Commit message: modify footprint
Parts:
- J2: footprint Connector_PinSocket_1.27mm:PinSocket_2x03_P1.27mm_Horizontal -> atmel_ice_adapter:PinSocket_2x03_P1.27mm_Horizontal
- J3: footprint Connector_PinSocket_2.54mm:PinSocket_2x03_P2.54mm_Horizontal -> atmel_ice_adapter:PinSocket_2x03_P2.54mm_Horizontal
- J4: footprint Connector_PinSocket_2.54mm:PinSocket_2x05_P2.54mm_Horizontal -> atmel_ice_adapter:PinSocket_2x05_P2.54mm_Horizontal
- J5: footprint Connector_PinSocket_2.54mm:PinSocket_2x10_P2.54mm_Horizontal -> atmel_ice_adapter:PinSocket_2x10_P2.54mm_Horizontal
Other:
- board text added: "-"
- board text added: "JLCJLCJLCJLC"
